File: pcb/PiHat_v2/RP4Hat/RP4Hat.kicad_sch (KiCad schematic)
At the start: 37 parts, among them J1 Conn_01x04, J2 Conn_01x04, J3 Conn_01x04, J4 Conn_01x04, J5 Conn_01x02, J6 Raspberry_Pi_4, J7 Conn_01x08, U1 THVD1410, U2 AP2112K-3.3

Commit message: new stuff.....
Other:
- added sheet LinearRegulator (LinearRegulator.kicad_sch)
- note added: "Linear Regulator"
Changed lines of the file:
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@@
 	(generator_version "9.0")
 	(paper "A4")
+	(text "Linear Regulator\n"
+		(exclude_from_sim no)
+		(at 184.15 107.442 0)
+		(effects
+			(font
+				(size 1.27 1.27)
+			)
+		)
+	)
 	(text "MAGNETIC ENCODER CONNECTORS"
 		(exclude_from_sim no)
@@
 				)
 			)
+		)
+	)
+	(sheet
+		(at 219.964 122.936)
+		(size 16.002 12.192)
+		(exclude_from_sim no)
+		(in_bom yes)
+		(on_board yes)
+		(dnp no)
+		(fields_autoplaced yes)
+		(stroke
+			(width 0.1524)
+			(type solid)
+		)
+		(fill
+			(color 0 0 0 0.0000)
+		)
+		(property "Sheetname" "LinearRegulator"
+			(at 219.964 122.2244 0)
+			(effects
+				(font
+					(size 1.27 1.27)
+				)
+				(justify left bottom)
+			)
+		)
+		(property "Sheetfile" "LinearRegulator.kicad_sch"
+			(at 219.964 135.7126 0)
+			(effects
+				(font
+					(size 1.27 1.27)
+				)
+				(justify left top)
+			)
+		)
+		(instances
+			(project "RP4Hat"
+				(path "/48e8712f-9e83-40b5-843b-6f1e3e03f403"
+					(page "2")
+				)
+			)
