File: pcb/PiHat_v3/RP4Hat/RP4Hat.kicad_pcb (KiCad board)
At the start: 4 copper layers, 65.6 x 56.6 mm, 38 parts, among them J1 Conn_01x04, J2 Conn_01x04, J3 Conn_01x04, J4 Conn_01x04, J5 Conn_01x02, J6 Raspberry_Pi_4, J7 Conn_01x08, U1 THVD1410, U2 AP2112K-3.3

Commit message: big potato shi
Parts:
- removed C1, C2, C3: 1uF, Capacitor_SMD:C_0805_2012Metric_Pad1.18x1.45mm_HandSolder
- removed G***: LOGO, LOGO
- removed J3, J4: Conn_01x04, Connector_JST:JST_PH_S4B-PH-K_1x04_P2.00mm_Horizontal
- removed J7: Conn_01x08, Connector_JST:JST_PH_S8B-PH-K_1x08_P2.00mm_Horizontal
- removed R14: 10k, Resistor_SMD:R_0805_2012Metric_Pad1.20x1.40mm_HandSolder
- removed R3, R4, R5, R6, R7: 100, Resistor_SMD:R_0805_2012Metric_Pad1.20x1.40mm_HandSolder
- added C14: 1uF, Capacitor_SMD:C_0805_2012Metric_Pad1.18x1.45mm_HandSolder, F.Cu at (73.9, 109.8)
- added C15: 1uF, Capacitor_SMD:C_0805_2012Metric_Pad1.18x1.45mm_HandSolder, F.Cu at (75.2, 83.4)
- added C16: 1uF, Capacitor_SMD:C_0805_2012Metric_Pad1.18x1.45mm_HandSolder, F.Cu at (77.1, 129.5)
- added C17: 22uF, Capacitor_SMD:C_1206_3216Metric_Pad1.33x1.80mm_HandSolder, F.Cu at (69.7, 139.3)
- added C9: 1uF, Capacitor_SMD:C_0805_2012Metric_Pad1.18x1.45mm_HandSolder, F.Cu at (55.2, 124.5)
- added J10: Conn_01x04, Connector_JST:JST_PH_S4B-PH-K_1x04_P2.00mm_Horizontal, F.Cu at (96.9, 87.2)
- added J11: Conn_01x02, Connector_JST:JST_PH_S2B-PH-K_1x02_P2.00mm_Horizontal, F.Cu at (67.2, 75.5)
- added J8: Conn_01x04, Connector_JST:JST_PH_S4B-PH-K_1x04_P2.00mm_Horizontal, F.Cu at (75.1, 87.2)
- added J9: Conn_01x04, Connector_JST:JST_PH_S4B-PH-K_1x04_P2.00mm_Horizontal, F.Cu at (86.0, 87.2)
- added R15: 100, Resistor_SMD:R_0805_2012Metric_Pad1.20x1.40mm_HandSolder, F.Cu at (77.1, 83.4)
- added R16: 100, Resistor_SMD:R_0805_2012Metric_Pad1.20x1.40mm_HandSolder, F.Cu at (79.0, 83.4)
- added R17: 100, Resistor_SMD:R_0805_2012Metric_Pad1.20x1.40mm_HandSolder, F.Cu at (88.0, 83.5)
- added R18: 100, Resistor_SMD:R_0805_2012Metric_Pad1.20x1.40mm_HandSolder, F.Cu at (90.0, 83.5)
- added R19: 100, Resistor_SMD:R_0805_2012Metric_Pad1.20x1.40mm_HandSolder, F.Cu at (99.0, 83.4)
- added R20: 100, Resistor_SMD:R_0805_2012Metric_Pad1.20x1.40mm_HandSolder, F.Cu at (100.9, 83.4)
- C11, C6, R1: moved to F.Cu
- C20, C4, U2: moved to B.Cu
- J2: value Conn_01x04 -> Conn_01x06; footprint Connector_JST:JST_PH_S4B-PH-K_1x04_P2.00mm_Horizontal -> Connector_JST:JST_PH_S6B-PH-K_1x06_P2.00mm_Horizontal
- R2: value 100 -> 10k
- U1: value THVD1410 -> ST3485ECDR; moved to F.Cu
- moved U1 93.1 mm to (52.3, 141.0), turned to 0 degrees
- moved R1 91.2 mm to (58.9, 142.1), turned to 0 degrees
- moved C6 84.5 mm to (58.9, 139.2), turned to 0 degrees
- moved C11 65.2 mm to (69.1, 124.5)
- moved J1 57.7 mm to (51.0, 130.4), turned to 0 degrees
- moved R2 44.9 mm to (73.9, 124.5), turned to 0 degrees
- moved R11 37.5 mm to (47.0, 78.6)
- moved R9 33.0 mm to (39.4, 79.0)
- moved R8 33.0 mm to (36.9, 79.0)
- moved R10 33.0 mm to (44.5, 78.7)
- moved R12 32.9 mm to (49.6, 78.6)
- moved J2 32.8 mm to (107.8, 87.2)
- moved R13 28.3 mm to (52.2, 78.6)
- moved C12 25.4 mm to (70.2, 70.0)
- moved C5 25.4 mm to (72.4, 69.9)
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Connections:
- net /A1 renamed /TW1_A
- net /A2 renamed /TW2_A
- net /B0 renamed /TW0_B
- A1 pad 1: /A0 -> /TW0_A
- A1 pad 11: /MISO -> /IMU0_MISO
- A1 pad 12: /CS -> /IMU0_CS
- A1 pad 14: /SCK -> /IMU0_SCK
- A1 pad 15: /MOSI -> /IMU0_MOSI
- A1 pad 29: /INT -> unconnected-(A1-GPIO22-Pad29)_1
- A1 pad 5: /B1 -> /TW1_B
- A1 pad 7: /B2 -> /TW2_B
- J2 pad 2: Net-(J2-Pin_2) -> /IMU0_MISO
- J2 pad 3: Net-(J2-Pin_3) -> /IMU0_MOSI
- J2 pad 4: GND -> /IMU0_SCK
- R11 pad 1: /B2 -> /TW1_B
- R13 pad 1: /B1 -> /TW2_B
- R2 pad 1: Net-(J2-Pin_2) -> +3.3V
- R2 pad 2: /A0 -> /IMU0_CS
- R8 pad 1: /A0 -> /TW0_A
Routing:
- net /EN: track 55.5 -> 0.00 mm
- net /A: track 55.5 -> 0.00 mm
- net /B: track 50.8 -> 0.00 mm
- net /RSTX: track 49.3 -> 0.00 mm
- net GND: track 50.0 -> 1.33 mm, vias 24 -> 1
- net /INT: track 47.2 -> 0.00 mm
- net /RSRX: track 40.6 -> 0.00 mm
- net /CS: track 38.8 -> 0.00 mm
- net /PICOTX: track 37.0 -> 0.00 mm
- net /PICORX: track 36.8 -> 0.00 mm
- net /SCK: track 30.3 -> 0.00 mm
- net /MISO: track 27.6 -> 0.00 mm
- net +5V: track 29.8 -> 4.56 mm, vias 9 -> 0
- net /MOSI: track 24.8 -> 0.00 mm
- net /TW0_A: track 0.00 -> 24.2 mm
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- added copper zone on B.Cu, net +3.3V
- removed copper zone on In2.Cu, net +3.3V
Other:
- outline, holes or cut-outs redrawn
- board text added: "IN"
- board text added: "OUT"
- board text removed: "GATR2"
- board text removed: "PI Hat V1 7/23"

Commit message: add supporting docs
Parts:
- U1: moved to B.Cu
- moved U1 119.6 mm to (122.2, 43.9)
- moved J1 111.8 mm to (128.1, 49.4), turned to 90 degrees
- moved C20 3.85 mm to (119.0, 75.7), turned to 180 degrees
- moved U2 3.33 mm to (122.6, 76.8)
- moved C4 3.33 mm to (122.5, 79.8)
- moved C5 0.61 mm to (73.0, 69.9)
- moved C12 0.60 mm to (70.8, 70.0)
- moved J11 0.55 mm to (67.8, 75.4)
- moved J5 0.55 mm to (67.8, 68.5)
Routing:
- net /TW2_A: track 0.00 -> 28.0 mm
- net /TW2_B: track 0.00 -> 27.8 mm
- net /TW1_A: track 0.00 -> 25.6 mm
- net /TW1_B: track 0.00 -> 25.4 mm
- net GND: track 1.33 -> 6.49 mm, vias 1 -> 4
- net Net-(J10-Pin_2): track 0.00 -> 2.79 mm
- net Net-(J10-Pin_3): track 0.00 -> 2.76 mm
- net Net-(J9-Pin_3): track 0.00 -> 2.74 mm
- net Net-(J9-Pin_2): track 0.00 -> 2.73 mm
- net +5V: track 4.56 -> 2.33 mm
