File: pcb/PiHat/PiHat_V3/RP4Hat/SPI_IMU.kicad_sch (KiCad schematic)
At the start: 3 parts, among them J2 Conn_01x06

Commit message: pcb changes
Connections:
- net CS: now also J2.4 (Pin_4); no longer J2.5 (Pin_5)
- net MISO: now also J2.5 (Pin_5); no longer J2.2 (Pin_2)
- net MOSI: now also J2.2 (Pin_2); no longer J2.3 (Pin_3)
- net SCK: now also J2.3 (Pin_3); no longer J2.4 (Pin_4)
Changed lines of the file:
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@@
 		)
 	)
-	(hierarchical_label "MOSI"
+	(hierarchical_label "SCK"
 		(shape input)
 		(at 135.89 95.25 0)
@@
 		)
 	)
-	(hierarchical_label "MISO"
+	(hierarchical_label "MOSI"
 		(shape input)
 		(at 135.89 92.71 0)
@@
 		)
 	)
-	(hierarchical_label "SCK"
+	(hierarchical_label "CS"
 		(shape input)
 		(at 135.89 97.79 0)
@@
 		)
 	)
-	(hierarchical_label "CS"
+	(hierarchical_label "MISO"
 		(shape input)
 		(at 135.89 100.33 0)
